File: cad/quadcopter/quadcopter.kicad_sch (KiCad schematic)
At the start: 41 parts, among them U1 8pin_header, U10 RQ5E040AJTCL, U11 2pin_header, U12 2pin_header, U13 LE33CZ-TR, U2 3pin_header, U3 Rust_Board, U4 2pin_header, U5 RQ5E040AJTCL, U6 RQ5E040AJTCL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

Commit message: Added several boards
Signed-off-by: Andrew Wock <ajwock@gmail.com>
Parts:
- C3, C4: footprint Imported:GCM033C70J104KE02D -> Capacitor_SMD:C_0603_1608Metric_Pad1.08x0.95mm_HandSolder
- R1, R11, R12, R13, R14, R2, R3, R4: footprint Resistor_SMD:R_0201_0603Metric -> Resistor_SMD:R_0603_1608Metric
Connections:
- net +BATT: now also C2.1; no longer C2.2
- net GND: now also C2.2; no longer C2.1
Other:
- moved on the sheet: C2, U4
