File: cad/quad_unibody/quad_unibody.kicad_pcb (KiCad board)
At the start: 2 copper layers, 63.5 x 55.9 mm, 64 parts, among them SW1 SW_Push, SW2 SW_Push, U1 LTC3534EGN#PBF, U10 2pin_header, U11 2pin_header, U12 3pin_header, U13 2pin_header, U14 ICM-42670-P, U2 ESP32-C3-MINI-1-H4X, U3 4pin_header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

Commit message: Big progress saver
Signed-off-by: Andrew Wock <ajwock@gmail.com>
Parts:
- added R28: 10k, Resistor_SMD:R_0603_1608Metric, F.Cu at (149.1, 126.5)
- added R29: 10k, Resistor_SMD:R_0603_1608Metric, F.Cu at (150.6, 127.1)
- added R30: 10k, Resistor_SMD:R_0603_1608Metric, F.Cu at (157.2, 129.0)
- R1, R7: value R_US -> 10k
Connections:
- U2 pad 22: pwm_frontright -> IO8
- U2 pad 27: IO19_USB_D+ -> pwm_frontright
Routing:
- net IO8: track 0.00 -> 8.97 mm, vias 0 -> 2
- net pwm_frontright: track 19.0 -> 11.7 mm
- net IO4_SDA: track 3.24 -> 7.25 mm
- net IO5_SCL: track 3.11 -> 6.96 mm, vias 0 -> 2
- net GND: track 18.9 -> 15.5 mm, vias 31 -> 32
