File: cad/quad_unibody/quad_unibody.kicad_sch (KiCad schematic)
At the start: 64 parts, among them SW1 SW_Push, SW2 SW_Push, U1 LTC3534EGN#PBF, U10 2pin_header, U11 2pin_header, U12 3pin_header, U13 2pin_header, U14 ICM-42670-P, U2 ESP32-C3-MINI-1-H4X, U3 4pin_header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

Commit message: Big progress saver
Signed-off-by: Andrew Wock <ajwock@gmail.com>
Parts:
- added R28, R29, R30: 10k, Resistor_SMD:R_0603_1608Metric, symbol Device:R_US
- R1, R7: value R_US -> 10k
Connections:
- net IO19_USB_D+ is gone; now on net pwm_frontright: U2.27 (IO19)
- net +3V3: now also R28.1, R29.1, R30.1
- net IO4_SDA: now also R28.2
- net IO5_SCL: now also R29.2
- net pwm_frontright: no longer U2.22 (IO8)
- new net IO8: R30.2, U2.22 (IO8)
- no-connect marks 1 -> 15
