File: cad/quadcopter/quad_direct/quad_direct.kicad_sch (KiCad schematic)
At the start: 15 parts, among them SW1 SW_Push, SW2 SW_Push, U1 4pin_header, U2 8pin_header, U3 8pin_header, U4 3pin_header

Commit message: Big progress saver
Signed-off-by: Andrew Wock <ajwock@gmail.com>
Parts:
- removed U2, U3: 8pin_header, Imported:8-bb, symbol Homebrewed:8pin_header
- added C7: .1u, Capacitor_SMD:C_0603_1608Metric, symbol Device:C
- added D1: LED, LED_SMD:LED_0603_1608Metric_Pad1.05x0.95mm_HandSolder, symbol Device:LED
- added R3, R4: 10k, Resistor_SMD:R_0603_1608Metric, symbol Device:R_US
- added U2: esp32c3_boardout, Imported:esp32c3_boardout, symbol Homebrewed:esp32c3_boardout
- R1, R2: value R_US -> 10k
- renumbered 11 to 111
Connections:
- net +3V3: now also R4.1, U2.16 (+3V3)
- net GND: now also C7.1, D1.1 (K), U2.15 (gnd)
- net IO0: now also U2.1 (io0)
- net IO1: now also U2.2 (io1)
- net IO10: now also R3.2, U2.12 (io10)
- net IO18_USB_D-: now also U2.11 (io18_d-)
- net IO19_USB_D+: now also U2.10 (io19_d+)
- net IO2: now also U2.3 (io2)
- net IO3: now also U2.4 (io3)
- net IO4: now also U2.5 (io4)
- net IO5: now also U2.6 (io5)
- net IO6: now also U2.7 (io6)
- net IO7: now also U2.8 (io7)
- net IO8: now also R4.2, U2.14 (io8)
- net IO9_BOOT: now also C7.2, U2.13 (boot)
- net RESET: now also U2.9 (reset)
- new net: D1.2 (A), R3.1
