File: cad/quadcopter/quad_direct/quad_direct.kicad_pcb (KiCad board)
At the start: 2 copper layers, 22.9 x 36.8 mm, 15 parts, among them SW1 SW_Push, SW2 SW_Push, U1 4pin_header, U2 8pin_header, U3 8pin_header, U4 3pin_header

Commit message: Tweaks to quad_direct eval board
Signed-off-by: Andrew Wock <ajwock@gmail.com>
Routing:
- net UART_RX: track 19.1 -> 20.2 mm, vias 1 -> 2
- net RESET: track 45.1 -> 45.6 mm
- net GND: vias 31 -> 26
Changed lines of the file:
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@@
   (via (at 152.654 70.612) (size 0.8) (drill 0.4) (layers "F.Cu" "B.Cu") (net 1))
   (via (at 164.8085 65.024) (size 0.8) (drill 0.4) (layers "F.Cu" "B.Cu") (net 1))
-  (segment (start 164.8085 62.5465) (end 168.95 58.405) (width 0.25) (layer "B.Cu") (net 1))
+  (segment (start 168.95 58.405) (end 167.19 60.165) (width 0.25) (layer "B.Cu") (net 1))
   (segment (start 152.69 79.3) (end 152.69 70.648) (width 0.25) (layer "B.Cu") (net 1))
-  (segment (start 164.8085 65.024) (end 164.8085 62.5465) (width 0.25) (layer "B.Cu") (net 1))
+  (segment (start 167.19 63.5) (end 165.666 65.024) (width 0.25) (layer "B.Cu") (net 1))
   (segment (start 152.69 70.648) (end 152.654 70.612) (width 0.25) (layer "B.Cu") (net 1))
+  (segment (start 167.19 60.165) (end 167.19 63.5) (width 0.25) (layer "B.Cu") (net 1))
+  (segment (start 165.666 65.024) (end 164.8085 65.024) (width 0.25) (layer "B.Cu") (net 1))
   (segment (start 160.02 76.975) (end 160.350402 76.975) (width 0.25) (layer "F.Cu") (net 2))
   (segment (start 150.33 62.332) (end 150.33 57.95) (width 0.25) (layer "F.Cu") (net 2))
@@
   (segment (start 155.194 75.184) (end 155.194 73.666) (width 0.25) (layer "F.Cu") (net 5))
   (via (at 155.194 75.184) (size 0.8) (drill 0.4) (layers "F.Cu" "B.Cu") (net 5))
-  (segment (start 156.808 73.57) (end 155.194 75.184) (width 0.25) (layer "B.Cu") (net 5))
-  (segment (start 148.59 58.435) (end 156.808 66.653) (width 0.25) (layer "B.Cu") (net 5))
-  (segment (start 156.808 66.653) (end 156.808 73.57) (width 0.25) (layer "B.Cu") (net 5))
+  (segment (start 148.59 59.436) (end 156.972 67.818) (width 0.25) (layer "B.Cu") (net 5))
+  (segment (start 156.972 67.818) (end 156.972 73.406) (width 0.25) (layer "B.Cu") (net 5))
+  (segment (start 156.972 73.406) (end 155.194 75.184) (width 0.25) (layer "B.Cu") (net 5))
+  (segment (start 148.59 58.435) (end 148.59 59.436) (width 0.25) (layer "B.Cu") (net 5))
   (segment (start 156.083 72.517) (end 156.083 73.577) (width 0.25) (layer "F.Cu") (net 6))
   (segment (start 156.083 73.577) (end 156.02 73.64) (width 0.25) (layer "F.Cu") (net 6))
@@
   (segment (start 167.64 66.294) (end 167.64 62.255) (width 0.25) (layer "B.Cu") (net 15))
   (segment (start 164.752 68.74) (end 164.084 68.072) (width 0.25) (layer "F.Cu") (net 16))
+  (segment (start 167.2965 52.8165) (end 167.2965 65.545793) (width 0.25) (layer "F.Cu") (net 16))
   (segment (start 165.92 68.74) (end 164.752 68.74) (width 0.25) (layer "F.Cu") (net 16))
+  (segment (start 167.2965 65.545793) (end 166.910326 65.931967) (width 0.25) (layer "F.Cu") (net 16))
+  (segment (start 166.55 52.07) (end 167.2965 52.8165) (width 0.25) (layer "F.Cu") (net 16))
   (via (at 164.084 68.072) (size 0.8) (drill 0.4) (layers "F.Cu" "B.Cu") (net 16))
-  (segment (start 164.084 68.072) (end 164.084 54.536) (width 0.25) (layer "B.Cu") (net 16))
-  (segment (start 164.084 54.536) (end 166.55 52.07) (width 0.25) (layer "B.Cu") (net 16))
+  (via (at 166.910326 65.931967) (size 0.8) (drill 0.4) (layers "F.Cu" "B.Cu") (net 16))
+  (segment (start 166.910326 65.931967) (end 164.770293 68.072) (width 0.25) (layer "B.Cu") (net 16))
+  (segment (start 164.770293 68.072) (end 164.084 68.072) (width 0.25) (layer "B.Cu") (net 16))
   (segment (start 166.57 67.94) (end 167.863 66.647) (width 0.25) (layer "F.Cu") (net 17))
   (segment (start 167.863 63.023) (end 168.854 62.032) (width 0.25) (layer "F.Cu") (net 17))
@@
   (via (at 163.957 81.407) (size 0.8) (drill 0.4) (layers "F.Cu" "B.Cu") (free) (net 19))
   (via (at 164.211 75.057) (size 0.8) (drill 0.4) (layers "F.Cu" "B.Cu") (free) (net 19))
-  (via (at 165.1 60.96) (size 0.8) (drill 0.4) (layers "F.Cu" "B.Cu") (free) (net 19))
   (via (at 154.178 73.787) (size 0.8) (drill 0.4) (layers "F.Cu" "B.Cu") (net 19))
   (via (at 156.591 83.82) (size 0.8) (drill 0.4) (layers "F.Cu" "B.Cu") (free) (net 19))
@@
   (via (at 156.718 75.184) (size 0.8) (drill 0.4) (layers "F.Cu" "B.Cu") (free) (net 19))
   (via (at 153.797 81.407) (size 0.8) (drill 0.4) (layers "F.Cu" "B.Cu") (free) (net 19))
-  (via (at 161.925 60.96) (size 0.8) (drill 0.4) (layers "F.Cu" "B.Cu") (free) (net 19))
   (via (at 148.209 77.978) (size 0.8) (drill 0.4) (layers "F.Cu" "B.Cu") (free) (net 19))
-  (via (at 167.005 59.055) (size 0.8) (drill 0.4) (layers "F.Cu" "B.Cu") (free) (net 19))
-  (via (at 166.116 62.484) (size 0.8) (drill 0.4) (layers "F.Cu" "B.Cu") (free) (net 19))
+  (via (at 157.988 64.008) (size 0.8) (drill 0.4) (layers "F.Cu" "B.Cu") (free) (net 19))
   (via (at 161.036 69.723) (size 0.8) (drill 0.4) (layers "F.Cu" "B.Cu") (free) (net 19))
-  (via (at 152.908 60.96) (size 0.8) (drill 0.4) (layers "F.Cu" "B.Cu") (free) (net 19))
-  (via (at 159.258 60.96) (size 0.8) (drill 0.4) (layers "F.Cu" "B.Cu") (free) (net 19))
+  (via (at 151.13 70.866) (size 0.8) (drill 0.4) (layers "F.Cu" "B.Cu") (free) (net 19))
   (via (at 166.243 77.216) (size 0.8) (drill 0.4) (layers "F.Cu" "B.Cu") (free) (net 19))
   (via (at 166.37 81.407) (size 0.8) (drill 0.4) (layers "F.Cu" "B.Cu") (free) (net 19))
-  (via (at 167.259 61.341) (size 0.8) (drill 0.4) (layers "F.Cu" "B.Cu") (free) (net 19))
   (via (at 163.957 77.216) (size 0.8) (drill 0.4) (layers "F.Cu" "B.Cu") (free) (net 19))
   (via (at 163.957 83.82) (size 0.8) (drill 0.4) (layers "F.Cu" "B.Cu") (free) (net 19))
   (via (at 149.733 53.594) (size 0.8) (drill 0.4) (layers "F.Cu" "B.Cu") (free) (net 19))
   (via (at 153.67 83.82) (size 0.8) (drill 0.4) (layers "F.Cu" "B.Cu") (free) (net 19))
-  (via (at 156.464 60.96) (size 0.8) (drill 0.4) (layers "F.Cu" "B.Cu") (free) (net 19))
+  (via (at 161.29 64.008) (size 0.8) (drill 0.4) (layers "F.Cu" "B.Cu") (free) (net 19))
   (via (at 156.718 81.407) (size 0.8) (drill 0.4) (layers "F.Cu" "B.Cu") (free) (net 19))
   (via (at 166.497 75.057) (size 0.8) (drill 0.4) (layers "F.Cu" "B.Cu") (free) (net 19))
@@
     )
   )
+  (zone (net 0) (net_name "") (layer "F.Cu") (hatch edge 0.508)
+    (connect_pads (clearance 0))
+    (min_thickness 0.254)
+    (keepout (tracks not_allowed) (vias not_allowed) (pads not_allowed) (copperpour not_allowed) (footprints allowed))
+    (fill (thermal_gap 0.508) (thermal_bridge_width 0.508))
+    (polygon
+      (pts
+        (xy 166.624 63.246)
+        (xy 153.416 63.246)
+        (xy 153.416 57.658)
+        (xy 166.624 57.658)
+      )
+    )
+  )
   (zone (net 19) (net_name "GND") (layer "B.Cu") (hatch edge 0.508)
     (connect_pads (clearance 0.508))
@@
       )
     )
+  )
+  (zone (net 0) (net_name "") (layer "B.Cu") (hatch edge 0.508)
+    (connect_pads (clearance 0))
+    (min_thickness 0.254)
+    (keepout (tracks not_allowed) (vias not_allowed) (pads not_allowed) (copperpour not_allowed) (footprints allowed))
+    (fill (thermal_gap 0.508) (thermal_bridge_width 0.508))
+    (polygon
+      (pts
+        (xy 153.416 63.246)
+        (xy 166.624 63.246)
+        (xy 166.624 57.658)
+        (xy 153.416 57.658)
+      )
+    )

Commit message: Big progress saver
Signed-off-by: Andrew Wock <ajwock@gmail.com>
Parts:
- removed 11: ESP32-C3-MINI-1-H4X, Imported:ESP32C3MINI1H4X
- removed U3: 8pin_header, Imported:8-bb
- added 111: ESP32-C3-MINI-1-H4X, Imported:ESP32C3MINI1H4X, F.Cu at (165.1, 35.6)
- added C7: .1u, Capacitor_SMD:C_0603_1608Metric, F.Cu at (168.3, 55.2)
- added D1: LED, LED_SMD:LED_0603_1608Metric_Pad1.05x0.95mm_HandSolder, F.Cu at (161.3, 48.9)
- added R3: 10k, Resistor_SMD:R_0603_1608Metric, F.Cu at (162.8, 46.5)
- added R4: 10k, Resistor_SMD:R_0603_1608Metric, F.Cu at (166.8, 46.5)
- R1, R2: value R_US -> 10k
- U2: value 8pin_header -> esp32c3_boardout; footprint Imported:8-bb -> Imported:esp32c3_boardout
- moved C3 33.7 mm to (157.2, 35.6), turned to 90 degrees
- moved R1 30.4 mm to (163.5, 54.1), turned to 180 degrees
- moved C2 30.2 mm to (155.5, 35.6)
- moved SW1 29.8 mm to (162.8, 57.8), turned to -90 degrees
- moved SW2 29.5 mm to (172.1, 57.8), turned to -90 degrees
- moved C6 28.6 mm to (160.2, 54.1), turned to 180 degrees
- moved R2 25.6 mm to (168.3, 53.5), turned to 0 degrees
- moved C1 24.8 mm to (156.4, 38.1), turned to 0 degrees
- moved U2 20.9 mm to (152.4, 63.5), turned to 0 degrees
- moved U1 18.9 mm to (175.3, 39.3), turned to 90 degrees
- moved C5 16.4 mm to (168.6, 51.5)
- moved U4 15.8 mm to (164.0, 49.0)
- moved C4 14.3 mm to (163.5, 51.5)
Connections:
- U2 pad 1: +3V3 -> IO0
- U2 pad 2: GND -> IO1
- U2 pad 3: IO8 -> IO2
- U2 pad 4: IO9_BOOT -> IO3
- U2 pad 5: IO10 -> IO4
- U2 pad 6: IO18_USB_D- -> IO5
- U2 pad 7: IO19_USB_D+ -> IO6
- U2 pad 8: RESET -> IO7
Routing:
- net GND: track 30.7 -> 1.61 mm, vias 26 -> 28
- net IO0: track 22.5 -> 5.84 mm, vias 1 -> 0
- net UART_RX: track 20.2 -> 6.08 mm, vias 2 -> 0
- net IO8: track 7.38 -> 20.4 mm
- net UART_TX: track 18.8 -> 7.71 mm
- net IO7: track 17.6 -> 28.1 mm
- net IO6: track 15.9 -> 25.1 mm
- net IO3: track 6.98 -> 15.7 mm
- net +3V3: track 61.7 -> 53.1 mm, vias 3 -> 2
- net +5V: track 17.3 -> 25.5 mm, vias 2 -> 1
- net IO1: track 15.7 -> 7.84 mm, vias 1 -> 0
- net IO10: track 13.6 -> 20.5 mm, vias 1 -> 4
- net IO5: track 15.8 -> 22.1 mm
- net IO19_USB_D+: track 13.0 -> 8.19 mm, vias 1 -> 0
- net IO2: track 10.1 -> 14.8 mm, vias 1 -> 0
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Other:
- board size 22.9 x 36.8 mm -> 24.1 x 40.1 mm

Commit message: Makera setup
Signed-off-by: Andrew Wock <ajwock@gmail.com>
Routing:
- net RESET: track 44.5 -> 63.4 mm, vias 3 -> 2
- net IO9_BOOT: track 28.1 -> 35.6 mm, vias 0 -> 2
- net +3V3: track 53.1 -> 46.1 mm
- net IO3: track 15.7 -> 18.3 mm, vias 1 -> 0
- net GND: track 1.61 -> 0.00 mm, vias 28 -> 7
- net IO6: track 25.1 -> 23.6 mm
- net IO7: track 28.1 -> 26.6 mm
- net IO5: track 22.1 -> 20.7 mm
- net IO2: track 14.8 -> 15.9 mm
- net IO4: track 19.1 -> 18.1 mm
- net +5V: track 25.5 -> 26.5 mm, vias 1 -> 0
- net IO10: track 20.5 -> 19.7 mm, vias 4 -> 3
- net IO8: vias 2 -> 0
Other:
- board size 24.1 x 40.1 mm -> 24.9 x 40.4 mm
