File: cad/quadcopter/quadcopter_boostbuck_small/quadcopter_boostbuck_small.kicad_pcb (KiCad board)
At the start: 2 copper layers, 25.4 x 10.2 mm, 14 parts, among them U1 3pin_header

Commit message: temp cad
Signed-off-by: Andrew Wock <ajwock@gmail.com>
Parts:
- moved C1 171.2 mm to (18.4, 18.3)
- moved C3 171.2 mm to (29.7, 21.3)
- moved C4 171.2 mm to (29.7, 19.8)
- moved C6 171.2 mm to (26.2, 23.5)
- moved R2 171.2 mm to (35.3, 21.9)
- moved R4 171.2 mm to (34.5, 19.4)
- moved R5 171.2 mm to (34.6, 17.4)
- moved U1 171.2 mm to (38.9, 22.8)
- moved 1 171.2 mm to (23.6, 19.7)
- moved C2 171.2 mm to (33.6, 21.9)
- moved C5 171.2 mm to (37.0, 18.7)
- moved L1 171.2 mm to (18.6, 21.6)
- moved R1 171.2 mm to (16.9, 18.9)
- moved R3 171.2 mm to (32.0, 20.4)
Routing:
- net GND: track 11.5 -> 1.84 mm
- net v_out: track 17.5 -> 17.0 mm
