File: cad/home_copter/home_copter.kicad_pcb (KiCad board)
At the start: 2 copper layers, 41.9 x 38.7 mm, 60 parts, among them U1 ICM-42670-P, U10 2pin_header, U11 2pin_header, U12 RQ5E040AJTCL, U13 RQ5E040AJTCL, U14 2pin_header, U15 2pin_header, U2 ESP32-C3-MINI-1-H4X, U3 LTC3534EGN#PBF, U4 USB3090-30-A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

Commit message: pre-homecopter change updates
Signed-off-by: Andrew Wock <ajwock@gmail.com>
Parts:
- removed REF** (x2): 0_ohm, Imported:0_ohm
- added C18: .1u, Capacitor_SMD:C_0603_1608Metric, F.Cu at (41.9, 32.3)
- added C2: 1u, Capacitor_SMD:C_0603_1608Metric, F.Cu at (27.7, 33.0)
- added C9: .1u, Capacitor_SMD:C_0603_1608Metric_Pad1.08x0.95mm_HandSolder, F.Cu at (65.8, 38.1)
- added D8: D_Schottky, Imported:SM6F22AY, F.Cu at (65.0, 32.3)
- added U16: 2pin_header, Imported:2-bb, F.Cu at (73.1, 25.1)
- added U17: 2pin_header, Imported:2-bb, F.Cu at (68.6, 28.7)
- added U5: 4pin_header, Imported:4-bb, F.Cu at (42.7, 17.7)
Connections:
- U4 pad 1: +BATT -> Net-(U4-Pad1)
Routing:
- net RESET: track 6.10 -> 10.4 mm
- net +3V3: track 111.7 -> 113.9 mm, vias 2 -> 5
- net IO9_BOOT: track 3.91 -> 5.91 mm

Commit message: Homecopter rev3
Signed-off-by: Andrew Wock <ajwock@gmail.com>
Parts:
- removed C3, C5: 470uF, Capacitor_THT:CP_Radial_D6.3mm_P2.50mm
- moved U16 47.7 mm to (26.7, 36.0), turned to -90 degrees
- moved C9 47.1 mm to (19.8, 27.9), turned to 180 degrees
- moved U17 27.0 mm to (42.5, 35.9), turned to -90 degrees
- moved D8 18.5 mm to (46.7, 34.8), turned to 180 degrees
- moved U5 8.13 mm to (42.7, 25.8)
- moved U6 6.93 mm to (23.8, 47.2)
- moved R18 5.78 mm to (42.9, 15.5)
- moved R20 5.78 mm to (42.9, 14.0)
- moved R19 4.49 mm to (39.6, 40.4)
- moved R21 4.49 mm to (39.6, 38.9)
- moved C15 2.93 mm to (37.8, 45.9)
- moved R10 2.93 mm to (40.8, 45.9)
- moved C12 2.93 mm to (39.3, 43.6)
- moved C13 2.93 mm to (37.8, 47.4)
- moved R13 2.93 mm to (41.9, 49.4)
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Routing:
- net UART_TX: track 0.00 -> 6.82 mm
- net Net-(U4-Pad1): track 0.00 -> 6.25 mm
- net UART_RX: track 0.00 -> 5.96 mm
- net Net-(R21-Pad2): track 1.56 -> 7.09 mm
- net Net-(R20-Pad2): track 1.71 -> 6.82 mm
- net +BATT: track 135.4 -> 138.2 mm
- net IO9_BOOT: track 5.91 -> 8.56 mm
- net RESET: track 10.4 -> 12.4 mm
- net pwm_backright: track 13.9 -> 12.0 mm
- net pwm_frontright: track 23.7 -> 21.8 mm
- net +3V3: track 113.9 -> 115.2 mm, vias 5 -> 3
- net IO18_USB_D+: track 5.09 -> 6.32 mm
- net IO18_USB_D-: track 5.03 -> 6.24 mm
- net GND: track 25.9 -> 26.9 mm, vias 12 -> 13
- net Net-(D6-Pad2): track 6.14 -> 6.97 mm
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