File: cad/home_copter/home_copter.kicad_sch (KiCad schematic)
At the start: 65 parts, among them U1 ICM-42670-P, U10 2pin_header, U11 2pin_header, U12 RQ5E040AJTCL, U13 RQ5E040AJTCL, U14 2pin_header, U15 2pin_header, U2 ESP32-C3-MINI-1-H4X, U3 LTC3534EGN#PBF, U4 USB3090-30-A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

Commit message: Homecopter rev3
Signed-off-by: Andrew Wock <ajwock@gmail.com>
Parts:
- gave numbers to parts that had none: 3
Changed lines of the file:
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@@
   (symbol (lib_id "Homebrewed:2pin_header") (at 152.4 35.56 0) (unit 1)
     (in_bom yes) (on_board yes)
-    (property "Reference" "U?" (id 0) (at 156.21 36.8299 0)
+    (property "Reference" "U16" (id 0) (at 156.21 36.8299 0)
       (effects (font (size 1.27 1.27)) (justify left))
     )
@@
   (symbol (lib_id "Homebrewed:2pin_header") (at 162.56 58.42 0) (unit 1)
     (in_bom yes) (on_board yes)
-    (property "Reference" "U?" (id 0) (at 166.37 59.6899 0)
+    (property "Reference" "U17" (id 0) (at 166.37 59.6899 0)
       (effects (font (size 1.27 1.27)) (justify left))
     )
@@
   (symbol (lib_id "Device:D_Schottky") (at 162.56 93.98 180) (unit 1)
     (in_bom yes) (on_board yes) (fields_autoplaced)
-    (property "Reference" "D?" (id 0) (at 162.8775 87.63 0))
+    (property "Reference" "D8" (id 0) (at 162.8775 87.63 0))
     (property "Value" "D_Schottky" (id 1) (at 162.8775 90.17 0))
     (property "Footprint" "Imported:SM6F22AY" (id 2) (at 162.56 93.98 0)
@@
     )
     (path "/973ca1d1-3d7c-4220-a222-8bdbdf7d33d7"
-      (reference "D?") (unit 1) (value "D_Schottky") (footprint "Imported:SM6F22AY")
+      (reference "D8") (unit 1) (value "D_Schottky") (footprint "Imported:SM6F22AY")
     )
     (path "/09f176d0-9833-4799-ae19-d9e810569567"
@@
     )
     (path "/62ba8ca4-b51e-4fee-b36c-ced3d3562acd"
-      (reference "U?") (unit 1) (value "2pin_header") (footprint "Imported:2-bb")
+      (reference "U16") (unit 1) (value "2pin_header") (footprint "Imported:2-bb")
     )
     (path "/7cdf64c9-c25f-4133-aab3-bc78ab414489"
-      (reference "U?") (unit 1) (value "2pin_header") (footprint "Imported:2-bb")
-    )
-  )
+      (reference "U17") (unit 1) (value "2pin_header") (footprint "Imported:2-bb")
+    )
+  )

Commit message: Likely hand solderable copter pcb finally designed!
Signed-off-by: Andrew Wock <ajwock@gmail.com>
Parts:
- U1: footprint Rust_Board:IC_ICM-42670-P -> Imported:ICM-42670-hand-solder
- U2: footprint Imported:ESP32C3MINI1H4X -> Imported:ESP32C3MINI1H4X_hand_solder
Changed lines of the file:
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@@
     (property "Reference" "U2" (id 0) (at 93.98 21.59 0))
     (property "Value" "ESP32-C3-MINI-1-H4X" (id 1) (at 93.98 24.13 0))
-    (property "Footprint" "Imported:ESP32C3MINI1H4X" (id 2) (at 68.58 34.29 0)
+    (property "Footprint" "Imported:ESP32C3MINI1H4X_hand_solder" (id 2) (at 68.58 34.29 0)
       (effects (font (size 1.27 1.27)) hide)
     )
@@
     (property "Reference" "U1" (id 0) (at 60.325 121.539 0))
     (property "Value" "ICM-42670-P" (id 1) (at 60.325 123.8504 0))
-    (property "Footprint" "Rust_Board:IC_ICM-42670-P" (id 2) (at 63.5 166.37 0)
+    (property "Footprint" "Imported:ICM-42670-hand-solder" (id 2) (at 63.5 166.37 0)
       (effects (font (size 1.27 1.27)) (justify left bottom) hide)
     )
@@
     )
     (path "/85e6dc1d-0713-44b3-8dee-438c88f0b01e"
-      (reference "U1") (unit 1) (value "ICM-42670-P") (footprint "Rust_Board:IC_ICM-42670-P")
+      (reference "U1") (unit 1) (value "ICM-42670-P") (footprint "Imported:ICM-42670-hand-solder")
     )
     (path "/608544e6-bb71-4ad0-a807-d7880397185b"
-      (reference "U2") (unit 1) (value "ESP32-C3-MINI-1-H4X") (footprint "Imported:ESP32C3MINI1H4X")
+      (reference "U2") (unit 1) (value "ESP32-C3-MINI-1-H4X") (footprint "Imported:ESP32C3MINI1H4X_hand_solder")
     )
     (path "/0bb91467-d5f3-4585-998c-8a1b79651589"
